Commit message: got axis_to_command_controller working, started on thruster_pid_controller

File: install/description/share/description/urdf/ROV2026.urdf.xacro (robot description, xacro)
@@ -1 +1,247 @@
-/home/artificer/Desktop/ROV2026/src/description/urdf/ROV2026.urdf.xacro
+<robot xmlns:xacro="http://ros.org/wiki/xacro" name="ROV2026">
+  <link name="base_link"/>
+  <xacro:macro name="thruster_control_joint" params="name">
+    <joint name="${name}_joint" type="continuous">
+      <command_interface name="effort"/>
+      <state_interface name="velocity"/>
+      <axis xyz="0 0 1"/>
+      <limit effort="1" velocity="100"/>
+    </joint>
+  </xacro:macro>
+  <ros2_control name="DummyHardwareSystem" type="system">
+    <hardware>
+      <plugin>dummy_hardware/DummyHardwareSystem</plugin>
+      <param name="pwm_freq_hz">50</param>
+      <param name="pwm_min_µs">1000</param>
+      <param name="pwm_max_µs">2000</param>
+      <param name="pwm_mid_µs">1500</param>
+    </hardware>
+    <xacro:thruster_control_joint name="front_left_bottom_thruster"/>
+    <xacro:thruster_control_joint name="front_right_bottom_thruster"/>
+    <xacro:thruster_control_joint name="front_left_top_thruster"/>
+    <xacro:thruster_control_joint name="front_right_top_thruster"/>
+    <xacro:thruster_control_joint name="back_left_bottom_thruster"/>
+    <xacro:thruster_control_joint name="back_right_bottom_thruster"/>
+    <xacro:thruster_control_joint name="back_left_top_thruster"/>
+    <xacro:thruster_control_joint name="back_right_top_thruster"/>
+  </ros2_control>
+  <!-- Thruster  Macro -->
+  <xacro:macro name="thruster" params="name x y z pitch yaw">
+    <!-- Link and Joint -->
+    <link name="${name}"/>
+    <joint name="${name}_joint" type="continuous">
+      <parent link="base_link"/>
+      <child link="${name}"/>
+      <origin
+        xyz="${float(x) * 0.01} ${float(y) * 0.01} ${float(z) * 0.01}"
+        rpy="
+        0
+        ${
+          float(pitch) * pi / 180.0
+        } ${
+          float(yaw) * pi / 180.0
+        }"
+      />
+      <axis xyz="0 0 1"/>
+      <limit effort="1" velocity="100"/>
+    </joint>
+  </xacro:macro>
+  <!--Ball Joint Macro-->
+  <xacro:macro name="ball_joint" params="name parent_link child_link x y z">
+    <!-- Intermediate links for the ball joint -->
+    <link name="${name}_x_link"/>
+    <link name="${name}_y_link"/>
+    <!-- Joints -->
+    <joint name="${name}_x_joint" type="revolute">
+      <parent link="${parent_link}"/>
+      <child link="${name}_x_link"/>
+      <origin xyz="${float(x) * 0.01} ${float(y) * 0.01} ${float(z) * 0.01}" rpy="0 0 0"/>
+      <axis xyz="1 0 0"/>
+      <limit lower="${-3/4 * pi}" upper="${3/4 * pi}" effort="5" velocity="5"/>
+    </joint>
+    <joint name="${name}_y_joint" type="revolute">
+      <parent link="${name}_x_link"/>
+      <child link="${name}_y_link"/>
+      <origin xyz="0 0 0" rpy="0 0 0"/>
+      <axis xyz="0 1 0"/>
+      <limit lower="${-3/4 * pi}" upper="${3/4 * pi}" effort="5" velocity="5"/>
+    </joint>
+    <joint name="${name}_z_joint" type="revolute">
+      <parent link="${name}_y_link"/>
+      <child link="${child_link}"/>
+      <origin xyz="0 0 0" rpy="0 0 0"/>
+      <axis xyz="0 0 1"/>
+      <limit lower="${-3/4 * pi}" upper="${3/4 * pi}" effort="5" velocity="5"/>
+    </joint>
+  </xacro:macro>
+  <!-- Linear Actuator-->
+  <xacro:macro name="linear_actuator" params="name parent_link child_link x y z lower upper">
+    <joint name="${name}_joint" type="prismatic">
+      <parent link="${parent_link}"/>
+      <child link="${child_link}"/>
+      <origin xyz="${float(x) * 0.01} ${float(y) * 0.01} ${float(z) * 0.01}" rpy="0 0 0"/>
+      <axis xyz="1 0 0"/> <!-- Point straight forward from the rpy direction -->
+      <limit lower="${float(actuator_distance) * -0.005}" upper="${float(actuator_distance) * 0.005}" effort="5" velocity="5"/>
+      <command_interface name="position"/>
+      <state_interface name="position"/>
+    </joint>
+  </xacro:macro>
+  <!-- Platform Connection Macro -->
+  <xacro:macro name="platform_connection" params="name parent_link child_link">
+    <joint name="${name}_joint" type="fixed">
+      <parent link="${parent_link}"/>
+      <child link="${child_link}"/>
+      <origin xyz="0 ${float(leg_length_upper) * 0.01} 0" rpy="0 0 0"/>
+    </joint>
+  </xacro:macro>
+  <!-- Thruster Properties -->
+  <xacro:property name="position_offset" value="16 30 16" />
+  <xacro:property name="rotation_offset" value="45 45" />
+  <!-- Thrusters -->
+  <xacro:thruster
+    name="front_left_bottom_thruster"
+    x="${-float(position_offset.split()[0])}"
+    y="${float(position_offset.split()[1])}"
+    z="${-float(position_offset.split()[2])}"
+    pitch="${-float(rotation_offset.split()[0])}"
+    yaw="${270 + float(rotation_offset.split()[1])}"
+  />
+  <xacro:thruster
+    name="front_right_bottom_thruster"
+    x="${float(position_offset.split()[0])}"
+    y="${float(position_offset.split()[1])}"
+    z="${-float(position_offset.split()[2])}"
+    pitch="${-float(rotation_offset.split()[0])}"
+    yaw="${float(rotation_offset.split()[1])}"
+  />
+  <xacro:thruster
+    name="front_left_top_thruster"
+    x="${-float(position_offset.split()[0])}"
+    y="${float(position_offset.split()[1])}"
+    z="${float(position_offset.split()[2])}"
+    pitch="${float(rotation_offset.split()[0])}"
+    yaw="${270 + float(rotation_offset.split()[1])}"
+  />
+  <xacro:thruster
+    name="front_right_top_thruster"
+    x="${float(position_offset.split()[0])}"
+    y="${float(position_offset.split()[1])}"
+    z="${float(position_offset.split()[2])}"
+    pitch="${float(rotation_offset.split()[0])}"
+    yaw="${float(rotation_offset.split()[1])}"
+  />
+  <xacro:thruster
+    name="back_left_bottom_thruster"
+    x="${-float(position_offset.split()[0])}"
+    y="${-float(position_offset.split()[1])}"
+    z="${-float(position_offset.split()[2])}"
+    pitch="${-float(rotation_offset.split()[0])}"
+    yaw="${180 + float(rotation_offset.split()[1])}"
+  />
+  <xacro:thruster
+    name="back_right_bottom_thruster"
+    x="${float(position_offset.split()[0])}"
+    y="${-float(position_offset.split()[1])}"
+    z="${-float(position_offset.split()[2])}"
+    pitch="${-float(rotation_offset.split()[0])}"
+    yaw="${90 + float(rotation_offset.split()[1])}"
+  />
+  <xacro:thruster
+    name="back_left_top_thruster"
+    x="${-float(position_offset.split()[0])}"
+    y="${-float(position_offset.split()[1])}"
+    z="${float(position_offset.split()[2])}"
+    pitch="${float(rotation_offset.split()[0])}"
+    yaw="${180 + float(rotation_offset.split()[1])}"
+  />
+  <xacro:thruster
+    name="back_right_top_thruster"
+    x="${float(position_offset.split()[0])}"
+    y="${-float(position_offset.split()[1])}"
+    z="${float(position_offset.split()[2])}"
+    pitch="${float(rotation_offset.split()[0])}"
+    yaw="${90 + float(rotation_offset.split()[1])}"
+  />
+  <!-- Arm Properties -->
+  <xacro:property name="legs_origin" value="0 0 0"/> <!-- x y z -->
+  <xacro:property name="leg_position_offset" value="4"/>
+  <xacro:property name="leg_length_lower" value="10"/>
+  <xacro:property name="leg_length_upper" value="3"/>
+  <xacro:property name="actuator_distance" value="20"/>
+  <xacro:linear_actuator
+    name="leg_actuator_1"
+    parent_link="base_link"
+    child_link="leg_shaft_lower_1"
+    x="${float(legs_origin.split()[0]) - (float(leg_position_offset) / sqrt(2))}"
+    y="${float(legs_origin.split()[1])}"
+    z="${float(legs_origin.split()[2]) + (float(leg_position_offset) / sqrt(2))}"
+    lower="${float(actuator_distance) / -2}"
+    upper="${float(actuator_distance) / 2}"
+  />
+  <xacro:linear_actuator
+    name="leg_actuator_2"
+    parent_link="base_link"
+    child_link="leg_shaft_lower_2"
+    x="${float(legs_origin.split()[0])}"
+    y="${float(legs_origin.split()[1])}"
+    z="${float(legs_origin.split()[2]) - float(leg_position_offset)}"
+    lower="${float(actuator_distance) / -2}"
+    upper="${float(actuator_distance) / 2}"
+  />
+  <xacro:linear_actuator
+    name="leg_actuator_3"
+    parent_link="base_link"
+    child_link="leg_shaft_lower_3"
+    x="${float(legs_origin.split()[0]) - (float(leg_position_offset) / sqrt(2))}"
+    y="${float(legs_origin.split()[1])}"
+    z="${float(legs_origin.split()[2]) + (float(leg_position_offset) / sqrt(2))}"
+    lower="${float(actuator_distance) / -2}"
+    upper="${float(actuator_distance) / 2}"
+  />
+  <link name="leg_shaft_lower_1"/>
+  <link name="leg_shaft_lower_2"/>
+  <link name="leg_shaft_lower_3"/>
+  <xacro:ball_joint
+    name="arm_joint_1"
+    parent_link="leg_shaft_lower_1"
+    child_link="leg_shaft_upper_1"
+    x="0"
+    y="${float(leg_length_lower) / 2}"
+    z="0"
+  />
+  <xacro:ball_joint
+    name="arm_joint_2"
+    parent_link="leg_shaft_lower_2"
+    child_link="leg_shaft_upper_2"
+    x="0"
+    y="${float(leg_length_lower) / 2}"
+    z="0"
+  />
+  <xacro:ball_joint
+    name="arm_joint_3"
+    parent_link="leg_shaft_lower_3"
+    child_link="leg_shaft_upper_3"
+    x="0"
+    y="${float(leg_length_lower) / 2}"
+    z="0"
+  />
+  <link name="leg_shaft_upper_1"/>
+  <link name="leg_shaft_upper_2"/>
+  <link name="leg_shaft_upper_3"/>
+  <link name="platform"/>
+  <xacro:platform_connection
+    name="leg_shaft_1_platform_connection"
+    parent_link="leg_shaft_upper_1"
+    child_link="platform"
+  />
+  <xacro:platform_connection
+    name="leg_shaft_2_platform_connection"
+    parent_link="leg_shaft_upper_2"
+    child_link="platform"
+  />
+  <xacro:platform_connection
+    name="leg_shaft_3_platform_connection"
+    parent_link="leg_shaft_upper_3"
+    child_link="platform"
+  />
+</robot>

Commit message: got everything working, started on depth/temp sensor

File: install/description/share/description/urdf/ROV2026.urdf.xacro (robot description, xacro)
@@ -1,247 +1 @@
-<robot xmlns:xacro="http://ros.org/wiki/xacro" name="ROV2026">
-  <link name="base_link"/>
-  <xacro:macro name="thruster_control_joint" params="name">
-    <joint name="${name}_joint" type="continuous">
-      <command_interface name="effort"/>
-      <state_interface name="velocity"/>
-      <axis xyz="0 0 1"/>
-      <limit effort="1" velocity="100"/>
-    </joint>
-  </xacro:macro>
-  <ros2_control name="DummyHardwareSystem" type="system">
-    <hardware>
-      <plugin>dummy_hardware/DummyHardwareSystem</plugin>
-      <param name="pwm_freq_hz">50</param>
-      <param name="pwm_min_µs">1000</param>
-      <param name="pwm_max_µs">2000</param>
-      <param name="pwm_mid_µs">1500</param>
-    </hardware>
-    <xacro:thruster_control_joint name="front_left_bottom_thruster"/>
-    <xacro:thruster_control_joint name="front_right_bottom_thruster"/>
-    <xacro:thruster_control_joint name="front_left_top_thruster"/>
-    <xacro:thruster_control_joint name="front_right_top_thruster"/>
-    <xacro:thruster_control_joint name="back_left_bottom_thruster"/>
-    <xacro:thruster_control_joint name="back_right_bottom_thruster"/>
-    <xacro:thruster_control_joint name="back_left_top_thruster"/>
-    <xacro:thruster_control_joint name="back_right_top_thruster"/>
-  </ros2_control>
-  <!-- Thruster  Macro -->
-  <xacro:macro name="thruster" params="name x y z pitch yaw">
-    <!-- Link and Joint -->
-    <link name="${name}"/>
-    <joint name="${name}_joint" type="continuous">
-      <parent link="base_link"/>
-      <child link="${name}"/>
-      <origin
-        xyz="${float(x) * 0.01} ${float(y) * 0.01} ${float(z) * 0.01}"
-        rpy="
-        0
-        ${
-          float(pitch) * pi / 180.0
-        } ${
-          float(yaw) * pi / 180.0
-        }"
-      />
-      <axis xyz="0 0 1"/>
-      <limit effort="1" velocity="100"/>
-    </joint>
-  </xacro:macro>
-  <!--Ball Joint Macro-->
-  <xacro:macro name="ball_joint" params="name parent_link child_link x y z">
-    <!-- Intermediate links for the ball joint -->
-    <link name="${name}_x_link"/>
-    <link name="${name}_y_link"/>
-    <!-- Joints -->
-    <joint name="${name}_x_joint" type="revolute">
-      <parent link="${parent_link}"/>
-      <child link="${name}_x_link"/>
-      <origin xyz="${float(x) * 0.01} ${float(y) * 0.01} ${float(z) * 0.01}" rpy="0 0 0"/>
-      <axis xyz="1 0 0"/>
-      <limit lower="${-3/4 * pi}" upper="${3/4 * pi}" effort="5" velocity="5"/>
-    </joint>
-    <joint name="${name}_y_joint" type="revolute">
-      <parent link="${name}_x_link"/>
-      <child link="${name}_y_link"/>
-      <origin xyz="0 0 0" rpy="0 0 0"/>
-      <axis xyz="0 1 0"/>
-      <limit lower="${-3/4 * pi}" upper="${3/4 * pi}" effort="5" velocity="5"/>
-    </joint>
-    <joint name="${name}_z_joint" type="revolute">
-      <parent link="${name}_y_link"/>
-      <child link="${child_link}"/>
-      <origin xyz="0 0 0" rpy="0 0 0"/>
-      <axis xyz="0 0 1"/>
-      <limit lower="${-3/4 * pi}" upper="${3/4 * pi}" effort="5" velocity="5"/>
-    </joint>
-  </xacro:macro>
-  <!-- Linear Actuator-->
-  <xacro:macro name="linear_actuator" params="name parent_link child_link x y z lower upper">
-    <joint name="${name}_joint" type="prismatic">
-      <parent link="${parent_link}"/>
-      <child link="${child_link}"/>
-      <origin xyz="${float(x) * 0.01} ${float(y) * 0.01} ${float(z) * 0.01}" rpy="0 0 0"/>
-      <axis xyz="1 0 0"/> <!-- Point straight forward from the rpy direction -->
-      <limit lower="${float(actuator_distance) * -0.005}" upper="${float(actuator_distance) * 0.005}" effort="5" velocity="5"/>
-      <command_interface name="position"/>
-      <state_interface name="position"/>
-    </joint>
-  </xacro:macro>
-  <!-- Platform Connection Macro -->
-  <xacro:macro name="platform_connection" params="name parent_link child_link">
-    <joint name="${name}_joint" type="fixed">
-      <parent link="${parent_link}"/>
-      <child link="${child_link}"/>
-      <origin xyz="0 ${float(leg_length_upper) * 0.01} 0" rpy="0 0 0"/>
-    </joint>
-  </xacro:macro>
-  <!-- Thruster Properties -->
-  <xacro:property name="position_offset" value="16 30 16" />
-  <xacro:property name="rotation_offset" value="45 45" />
-  <!-- Thrusters -->
-  <xacro:thruster
-    name="front_left_bottom_thruster"
-    x="${-float(position_offset.split()[0])}"
-    y="${float(position_offset.split()[1])}"
-    z="${-float(position_offset.split()[2])}"
-    pitch="${-float(rotation_offset.split()[0])}"
-    yaw="${270 + float(rotation_offset.split()[1])}"
-  />
-  <xacro:thruster
-    name="front_right_bottom_thruster"
-    x="${float(position_offset.split()[0])}"
-    y="${float(position_offset.split()[1])}"
-    z="${-float(position_offset.split()[2])}"
-    pitch="${-float(rotation_offset.split()[0])}"
-    yaw="${float(rotation_offset.split()[1])}"
-  />
-  <xacro:thruster
-    name="front_left_top_thruster"
-    x="${-float(position_offset.split()[0])}"
-    y="${float(position_offset.split()[1])}"
-    z="${float(position_offset.split()[2])}"
-    pitch="${float(rotation_offset.split()[0])}"
-    yaw="${270 + float(rotation_offset.split()[1])}"
-  />
-  <xacro:thruster
-    name="front_right_top_thruster"
-    x="${float(position_offset.split()[0])}"
-    y="${float(position_offset.split()[1])}"
-    z="${float(position_offset.split()[2])}"
-    pitch="${float(rotation_offset.split()[0])}"
-    yaw="${float(rotation_offset.split()[1])}"
-  />
-  <xacro:thruster
-    name="back_left_bottom_thruster"
-    x="${-float(position_offset.split()[0])}"
-    y="${-float(position_offset.split()[1])}"
-    z="${-float(position_offset.split()[2])}"
-    pitch="${-float(rotation_offset.split()[0])}"
-    yaw="${180 + float(rotation_offset.split()[1])}"
-  />
-  <xacro:thruster
-    name="back_right_bottom_thruster"
-    x="${float(position_offset.split()[0])}"
-    y="${-float(position_offset.split()[1])}"
-    z="${-float(position_offset.split()[2])}"
-    pitch="${-float(rotation_offset.split()[0])}"
-    yaw="${90 + float(rotation_offset.split()[1])}"
-  />
-  <xacro:thruster
-    name="back_left_top_thruster"
-    x="${-float(position_offset.split()[0])}"
-    y="${-float(position_offset.split()[1])}"
-    z="${float(position_offset.split()[2])}"
-    pitch="${float(rotation_offset.split()[0])}"
-    yaw="${180 + float(rotation_offset.split()[1])}"
-  />
-  <xacro:thruster
-    name="back_right_top_thruster"
-    x="${float(position_offset.split()[0])}"
-    y="${-float(position_offset.split()[1])}"
-    z="${float(position_offset.split()[2])}"
-    pitch="${float(rotation_offset.split()[0])}"
-    yaw="${90 + float(rotation_offset.split()[1])}"
-  />
-  <!-- Arm Properties -->
-  <xacro:property name="legs_origin" value="0 0 0"/> <!-- x y z -->
-  <xacro:property name="leg_position_offset" value="4"/>
-  <xacro:property name="leg_length_lower" value="10"/>
-  <xacro:property name="leg_length_upper" value="3"/>
-  <xacro:property name="actuator_distance" value="20"/>
-  <xacro:linear_actuator
-    name="leg_actuator_1"
-    parent_link="base_link"
-    child_link="leg_shaft_lower_1"
-    x="${float(legs_origin.split()[0]) - (float(leg_position_offset) / sqrt(2))}"
-    y="${float(legs_origin.split()[1])}"
-    z="${float(legs_origin.split()[2]) + (float(leg_position_offset) / sqrt(2))}"
-    lower="${float(actuator_distance) / -2}"
-    upper="${float(actuator_distance) / 2}"
-  />
-  <xacro:linear_actuator
-    name="leg_actuator_2"
-    parent_link="base_link"
-    child_link="leg_shaft_lower_2"
-    x="${float(legs_origin.split()[0])}"
-    y="${float(legs_origin.split()[1])}"
-    z="${float(legs_origin.split()[2]) - float(leg_position_offset)}"
-    lower="${float(actuator_distance) / -2}"
-    upper="${float(actuator_distance) / 2}"
-  />
-  <xacro:linear_actuator
-    name="leg_actuator_3"
-    parent_link="base_link"
-    child_link="leg_shaft_lower_3"
-    x="${float(legs_origin.split()[0]) - (float(leg_position_offset) / sqrt(2))}"
-    y="${float(legs_origin.split()[1])}"
-    z="${float(legs_origin.split()[2]) + (float(leg_position_offset) / sqrt(2))}"
-    lower="${float(actuator_distance) / -2}"
-    upper="${float(actuator_distance) / 2}"
-  />
-  <link name="leg_shaft_lower_1"/>
-  <link name="leg_shaft_lower_2"/>
-  <link name="leg_shaft_lower_3"/>
-  <xacro:ball_joint
-    name="arm_joint_1"
-    parent_link="leg_shaft_lower_1"
-    child_link="leg_shaft_upper_1"
-    x="0"
-    y="${float(leg_length_lower) / 2}"
-    z="0"
-  />
-  <xacro:ball_joint
-    name="arm_joint_2"
-    parent_link="leg_shaft_lower_2"
-    child_link="leg_shaft_upper_2"
-    x="0"
-    y="${float(leg_length_lower) / 2}"
-    z="0"
-  />
-  <xacro:ball_joint
-    name="arm_joint_3"
-    parent_link="leg_shaft_lower_3"
-    child_link="leg_shaft_upper_3"
-    x="0"
-    y="${float(leg_length_lower) / 2}"
-    z="0"
-  />
-  <link name="leg_shaft_upper_1"/>
-  <link name="leg_shaft_upper_2"/>
-  <link name="leg_shaft_upper_3"/>
-  <link name="platform"/>
-  <xacro:platform_connection
-    name="leg_shaft_1_platform_connection"
-    parent_link="leg_shaft_upper_1"
-    child_link="platform"
-  />
-  <xacro:platform_connection
-    name="leg_shaft_2_platform_connection"
-    parent_link="leg_shaft_upper_2"
-    child_link="platform"
-  />
-  <xacro:platform_connection
-    name="leg_shaft_3_platform_connection"
-    parent_link="leg_shaft_upper_3"
-    child_link="platform"
-  />
-</robot>
+/home/student/Desktop/ROV2026/src/description/urdf/ROV2026.urdf.xacro
